File: Motor.kicad_sch (KiCad schematic)
At the start: 117 parts, among them J13 POWER_UNO, J14 POWER_UNO, J15 POWER_UNO, J16 POWER_UNO, J17 ICSP, J18 ICSP, J19 ICSP, J20 ICSP, J21 ICSP, M1 DRV8305NQPHPRQ1, M2 DRV8305NQPHPRQ1, Q1 100V 6A, Q10 100V 6A, Q11 100V 6A, Q12 100V 6A, Q2 100V 6A, Q3 100V 6A, Q4 100V 6A, Q5 100V 6A, Q6 100V 6A, Q7 100V 6A, Q8 100V 6A, Q9 100V 6A

Commit message: Changes to layout pins
Parts:
- removed J13, J14, J15, J16: POWER_UNO, Header 8x1 8.5mm, symbol ISS_ALT_LIB:root_0_POWER_UNO_ISS_ALT_LIB.SchLib
- removed J17, J18, J19, J20, J21: ICSP, ICSP, symbol ISS_ALT_LIB:root_0_ICSP_ISS_ALT_LIB.SchLib
- removed R100, R101, R102, R109, R111, R113, R115, R117, R118, R119, R120, R74, R77, R78, R79, R81, R82, R83, R84, R92, R93, R95, R98, R99: 0R, RES_0603, symbol ISS_ALT_LIB:root_0_RES_0603_ISS_ALT_LIB.SchLib
- removed R110, R112, R114, R116, R73, R75, R76, R80, R91, R94, R96, R97: 10K, RES_0603, symbol ISS_ALT_LIB:root_0_RES_0603_ISS_ALT_LIB.SchLib
- added C190: .1uF, Capacitor_SMD:C_0402_1005Metric, symbol Device:C_Small
- added C191: 10uF, Capacitor_SMD:C_0603_1608Metric, symbol Device:C_Small
- added R110, R112, R114, R116, R73, R75, R76, R80, R91, R94, R96, R97: 10K, Resistor_SMD:R_0603_1608Metric, symbol Device:R
- added U24: MAX11128xTI, Package_DFN_QFN:TQFN-28-1EP_5x5mm_P0.5mm_EP3.25x3.25mm, symbol Analog_ADC:MAX11128xTI
- C101, C102, C107, C108, C113, C114, C85, C86, C91, C92: symbol ISS_ALT_LIB:root_3_CAP_0603_ISS_ALT_LIB.SchLib -> Device:C
- C105, C106, C111, C112, C116, C118, C89, C90: symbol ISS_ALT_LIB:root_1_CAP_0603_ISS_ALT_LIB.SchLib -> Device:C
- M1, M2: symbol RPOD_UPPR:root_0_DRV8305NQPHPRQ1_RPOD_UPPR.SchLib -> KiCAD_Library_Cooter:root_0_DRV8305NQPHPRQ1_RPOD_UPPR.SchLib
- Q1, Q10, Q11, Q12, Q2, Q3, Q4, Q5, Q6, Q7, Q8, Q9: footprint PMPB29XNEAX:TRANS_BUK9D23-40EX -> Library:UDFN6B; symbol ISS_ALT_LIB:root_0_SSM6K341NU,LF_ISS_ALT_LIB.SchLib -> KiCAD_Library_Cooter:root_0_SSM6K341NU,LF_ISS_ALT_LIB.SchLib
- R103, R104, R121, R122, R85, R86: footprint RES_0805 -> Resistor_SMD:R_0603_1608Metric; symbol ISS_ALT_LIB:root_1_RES_0805_ISS_ALT_LIB.SchLib -> Device:R
- R105, R106, R107, R108, R123, R124, R125, R126, R87, R88, R89, R90: footprint RES_0603 -> Resistor_SMD:R_0603_1608Metric; symbol ISS_ALT_LIB:root_1_RES_0603_ISS_ALT_LIB.SchLib -> Device:R
- R67, R68, R69, R70: footprint RES_0402 -> Resistor_SMD:R_0402_1005Metric
- R71, R72: footprint RES_0603 -> Resistor_SMD:R_0603_1608Metric; symbol ISS_ALT_LIB:root_0_RES_0603_ISS_ALT_LIB.SchLib -> Device:R
Connections:
- net ISNS_NA_MTR1 is gone; now on net GND: C102.2, M1.24 (SP1)
- net ISNS_NA_MTR2 is gone; now on net GND: C101.2, M2.24 (SP1)
- net ISNS_NB_MTR1 is gone; now on net GND: C108.2, M1.22 (SP2)
- net ISNS_NB_MTR2 is gone; now on net GND: C107.2, M2.22 (SP2)
- net ISNS_NC_MTR1 is gone; now on net GND: C114.2, M1.20 (SP3)
- net ISNS_NC_MTR2 is gone; now on net GND: C113.2, M2.20 (SP3)
- net SCLK_MTR2 is gone; now on net MTR_SCLK: M2.12 (SCLK)
- net SDI_MTR2 is gone; now on net MTR_SDI: M2.10 (SDI)
- net SDO_MTR2 is gone; now on net MTR_SDO: M2.11 (SDO)
- net SL_A_MTR1 is gone; now on net ISNS_PA_MTR1: M1.34 (SLA), Q4.4 (S_1), Q4.7 (S_2), R86.2
- net SL_A_MTR2 is gone; now on net ISNS_PA_MTR2: M2.34 (SLA), Q1.4 (S_1), Q1.7 (S_2), R85.2
- net SL_B_MTR1 is gone; now on net ISNS_PB_MTR1: M1.31 (SLB), Q8.4 (S_1), Q8.7 (S_2), R104.2
- net SL_B_MTR2 is gone; now on net ISNS_PB_MTR2: M2.31 (SLB), Q6.4 (S_1), Q6.7 (S_2), R103.2
- net SL_C_MTR1 is gone; now on net ISNS_PC_MTR1: M1.26 (SLC), Q11.4 (S_1), Q11.7 (S_2), R122.2
- net SL_C_MTR2 is gone; now on net ISNS_PC_MTR2: M2.26 (SLC), Q10.4 (S_1), Q10.7 (S_2), R121.2
- net GH_A_MTR1: now also Q3.3 (G), R75.1
- net GH_A_MTR2: now also Q2.3 (G), R76.1
- net GH_B_MTR1: now also Q7.3 (G), R94.1
- net GH_B_MTR2: now also Q5.3 (G), R97.1
- net GH_C_MTR1: now also Q12.3 (G), R112.1
- net GH_C_MTR2: now also Q9.3 (G), R114.1
- net GL_A_MTR1: now also Q4.3 (G), R73.1
- net GL_A_MTR2: now also Q1.3 (G), R80.1
- net GL_B_MTR1: now also Q8.3 (G), R96.1
- net GL_B_MTR2: now also Q6.3 (G), R91.1
- net GL_C_MTR1: now also Q11.3 (G), R116.1
- net GL_C_MTR2: now also Q10.3 (G), R110.1
- net GND: now also C190.2, C191.2, U24.14 (GND), U24.16 (GND), U24.22 (DGND), U24.29 (EP)
- net ISNS_PA_MTR1: now also R73.2
- net ISNS_PA_MTR2: now also R80.2
- net ISNS_PB_MTR1: now also R96.2
- net ISNS_PB_MTR2: now also R91.2
- net ISNS_PC_MTR1: now also R116.2
- net ISNS_PC_MTR2: now also R110.2
- net P3V3: now also C190.1, C191.1, U24.17 (VDD), U24.18 (VDD), U24.23 (OVDD)
- net ENGATE_MTR1 renamed MTR_WHA_EN
- net ENGATE_MTR2 renamed MTR_WHB_EN
- net INHA_MTR1 renamed MTR_WHA_INA_H
- net INHA_MTR2 renamed MTR_WHB_INA_H
- net INHB_MTR1 renamed MTR_WHA_INB_H
- net INHB_MTR2 renamed MTR_WHB_INB_H
- net INHC_MTR1 renamed MTR_WHA_INC_H
- net INHC_MTR2 renamed MTR_WHB_INC_H
- net INLA_MTR1 renamed MTR_WHA_INA_L
- net INLA_MTR2 renamed MTR_WHB_INA_L
- net INLB_MTR1 renamed MTR_WHA_INB_L
- net INLB_MTR2 renamed MTR_WHB_INB_L
- net INLC_MTR1 renamed MTR_WHA_INC_L
- net INLC_MTR2 renamed MTR_WHB_INC_L
- net MTR1_ISNS_A renamed MTR_WHA_iSEN_A
- net MTR_WHA_iSEN_A: now also U24.4 (AIN6)
- net MTR1_ISNS_B renamed MTR_WHA_iSEN_B
- net MTR_WHA_iSEN_B: now also U24.5 (AIN7)
- net MTR1_ISNS_C renamed MTR_WHA_iSEN_C
- net MTR_WHA_iSEN_C: now also U24.6 (AIN8)
- net MTR2_ISNS_A renamed MTR_WHB_iSEN_A
- net MTR_WHB_iSEN_A: now also U24.7 (AIN9)
- net MTR2_ISNS_B renamed MTR_WHB_iSEN_B
- net MTR_WHB_iSEN_B: now also U24.8 (AIN10)
- net MTR2_ISNS_C renamed MTR_WHB_iSEN_C
- net MTR_WHB_iSEN_C: now also U24.9 (AIN11)
- net NFLT_MTR1 renamed _MTR_WHA_nFAULT
- net NFLT_MTR2 renamed _MTR_WHB_nFAULT
- net NSCS_MTR1 renamed MTR_WHA_SCS
- net NSCS_MTR2 renamed MTR_WHB_SCS
- net PHA_MTR_1 renamed MTR_WHA_PHA
- net MTR_WHA_PHA: now also R75.2
- net PHA_MTR_2 renamed MTR_WHB_PHA
- net MTR_WHB_PHA: now also R76.2
- net PHB_MTR_1 renamed MTR_WHA_PHB
- net MTR_WHA_PHB: now also R94.2
- net PHB_MTR_2 renamed MTR_WHB_PHB
- net MTR_WHB_PHB: now also R97.2
- net PHC_MTR_1 renamed MTR_WHA_PHC
- net MTR_WHA_PHC: now also R112.2
- net PHC_MTR_2 renamed MTR_WHB_PHC
- net MTR_WHB_PHC: now also R114.2
- net SCLK_MTR1 renamed MTR_SCLK
- net SDI_MTR1 renamed MTR_SDI
- net SDO_MTR1 renamed MTR_SDO
- net VSNS_A_MTR1 renamed MTR_WHA_VSNS_A
- net MTR_WHA_VSNS_A: now also U24.1 (AIN3)
- net VSNS_A_MTR2 renamed MTR_WHB_VSNS_A
- net MTR_WHB_VSNS_A: now also U24.26 (AIN0)
- net VSNS_B_MTR1 renamed MTR_WHA_VSNS_B
- net MTR_WHA_VSNS_B: now also U24.27 (AIN1)
- net VSNS_B_MTR2 renamed MTR_WHB_VSNS_B
- net MTR_WHB_VSNS_B: now also U24.2 (AIN4)
- net VSNS_C_MTR1 renamed MTR_WHA_VSNS_C
- net MTR_WHA_VSNS_C: now also U24.3 (AIN5)
- net VSNS_C_MTR2 renamed MTR_WHB_VSNS_C
- net MTR_WHB_VSNS_C: now also U24.28 (AIN2)
- net WAKE_MTR_1 renamed MTR_WHA_WAKE
- net WAKE_MTR_2 renamed MTR_WHB_WAKE
- new net MOTOR_ADC_CS: U24.20 (~{CS})
- new net SPI1_MISO: U24.24 (DOUT)
- new net SPI1_MOSI: U24.21 (DIN)
- new net SPI1_SCLK: U24.19 (SCLK)
- no-connect marks 0 -> 5
Other:
- moved on the sheet: C100, C104, C109, C110, C115, C117, C87, C88, C94, C95, C96, C97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
