File: storage.kicad_sch (KiCad schematic)
At the start: 7 parts, among them J12 Micro_SD_Card, U8 S25FL256SAGNFI001

Commit message: Changes to layout pins
Connections:
- net GND: now also J12.SH (SHIELD); no longer J12.9 (SHIELD)
Changed lines of the file:
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@@
 		(pin "6"
 		)
-		(pin "9"
+		(pin "SH"
 		)
 		(instances
